File: vscp-din-wireless-esp8266-flat.sch (KiCad schematic (older format))
At the start: 24 parts, among them J1 Conn_01x04_Left, J2 Conn_01x04_Right, J3 Conn_01x06, J4 Conn_01x02, Q1 BC547, U2 ESP-12E

Commit message: Added gerbers
Parts:
- removed C6: 100nF, Capacitor_SMD:C_0805_2012Metric, symbol Device:C
- removed J1: Conn_01x04_Left, Connector_PinHeader_2.54mm:PinHeader_1x04_P2.54mm_Vertical, symbol Connector_Generic:Conn_01x04
- removed J2: Conn_01x04_Right, Connector_PinHeader_2.54mm:PinHeader_1x04_P2.54mm_Vertical, symbol Connector_Generic:Conn_01x04
- removed R12: 0R, Resistor_SMD:R_0805_2012Metric, symbol Device:R_Small
- added C4: 100nF, Capacitor_SMD:C_0805_2012Metric, symbol Device:C
- added J1: Conn_01x12, Connector_PinSocket_2.54mm:PinSocket_1x12_P2.54mm_Vertical, symbol Connector_Generic:Conn_01x12
Connections:
- net GND: now also C4.2, J1.12 (Pin_12)
- net VCC: now also J1.1 (Pin_1)
- net VDD: now also C4.1, J1.2 (Pin_2)
- net TTLRX: now reaches Q1.2 (B), R9.1
- net MISO: now reaches U2.10 (MISO)
- net MISO: now also J1.8 (Pin_8)
- net gpio9: now reaches U2.11 (GPIO9)
- net gpio9: now also J1.11 (Pin_11)
- net MOSI: now reaches U2.13 (MOSI)
- net MOSI: now also J1.9 (Pin_9)
- net SCLK: now reaches U2.14 (SCLK)
- net SCLK: now also J1.10 (Pin_10)
- net adc: now reaches U2.2 (ADC)
- net adc: now also J1.3 (Pin_3)
- net gpio14: now reaches U2.5 (GPIO14)
- net gpio14: now also J1.4 (Pin_4)
- net gpio12: now reaches U2.6 (GPIO12)
- net gpio12: now also J1.5 (Pin_5)
- net gpio13: now reaches U2.7 (GPIO13)
- net gpio13: now also J1.6 (Pin_6)
- net CS0: now reaches U2.9 (CS0)
- net CS0: now also J1.7 (Pin_7)
Other:
- moved on the sheet: C5
